File: class_AB_amplifier_opamp/class_AB_amplifier_opamp.kicad_pcb (KiCad board)
At the start: 2 copper layers, 90.2 x 50.8 mm, 23 parts, among them J1 Entrada de alimentación, J2 Entrada de Señal, J3 Salida de señal, Q1 TIP41, Q2 TIP42, U1 LM741

Commit message: pdfs esquematico y pcb
Parts:
- moved C4 9.86 mm to (55.9, 32.0)
- moved J1 9.86 mm to (24.1, 47.2)
- moved C1 9.86 mm to (26.7, 26.9)
- moved C3 9.86 mm to (95.2, 39.6)
- moved D2 9.86 mm to (34.3, 47.2)
- moved D3 9.86 mm to (101.6, 32.0)
- moved D4 9.86 mm to (94.0, 26.9)
- moved D5 9.86 mm to (67.3, 47.2)
- moved D6 9.86 mm to (59.7, 62.5)
- moved J2 9.86 mm to (47.0, 24.4)
- moved J3 9.86 mm to (52.1, 62.5)
- moved Q1 9.86 mm to (97.8, 62.5)
- moved Q2 9.86 mm to (74.9, 62.5)
- moved R1 9.86 mm to (74.9, 32.0)
- moved R2 9.86 mm to (64.8, 26.9)
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