File: tia+bfsk_demodulator/tia+bfsk_demodulator.kicad_sch (KiCad schematic)
At the start: 30 parts, among them U1 4046, U2 40106, U3 LM358, U4 LM358, U5 40106

Commit message: agrego amplificador clase AB
Parts:
- C10: value 100n -> 1n
Changed lines of the file:
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@@
       (effects (font (size 1.27 1.27)) (justify left))
     )
-    (property "Value" "100n" (at 120.65 54.61 90)
+    (property "Value" "1n" (at 120.65 54.61 90)
       (effects (font (size 1.27 1.27)) (justify left))
     )

Commit message: actualizo con proy td3
Parts:
- removed C4: 2.2n, symbol Device:C
- removed R4: 47k, symbol Device:R
- removed U2: 40106, symbol 4xxx_IEEE:40106
- added C11: 2p, symbol Device:C
- added C12: 2.2n, symbol Device:C
- added R14: 470k, symbol Device:R
- added R15, R16, R17: 10k, symbol Device:R
- added U6: 4050, symbol 4xxx:4050
- added U7: LM324, symbol Amplifier_Operational:LM324
- C1: value 2.2n -> 1n
- C6: value 100n -> 1n
- R3: value 47k -> 100k
Connections:
- net Demod: now also C11.2, R16.2, U7.1
- net GND: now also C12.1, R17.1
- net STM32 Input: now also U6.2
- net at C6.2, R6.2, R7.1: now also U6.3
- net at R3.1, U1.10 (SFout): now also R14.1
- new net: C11.1, C12.2, R14.2, R15.1
- new net: R16.1, R17.2, U7.2 (-)
- new net: R15.2, U7.3 (+)
Other:
- note added: "LPF must match to remove the high logic frequency (16KHz)"
- company: (none) -> Designer: Alan Vel
- title: (none) -> BFSK for VLC link
- moved on the sheet: C6, R3, R5, R6, R7, R8
