File: vlc_communication/vlc_communication.kicad_sch (KiCad schematic)
At the start: 107 parts, among them J1 Input 5V, J2 Motor, Q1 BC546, Q2 BC546, Q3 BC546, U1 4046, U10 40106, U11 4046, U12 LM324, U13 LM324, U2 LM324, U3 LM358, U4 LM358, U5 40106, U6 STM32F103C8Tx BLUEPILL, U7 LM324, U8 LM358, U9 LM358

Commit message: avances de proyecto
Parts:
- removed D5, D6: 1N4148, Diode_THT:D_DO-35_SOD27_P7.62mm_Horizontal, symbol Diode:1N4148
- removed U3, U4, U8, U9: LM358, symbol Amplifier_Operational:LM358
- removed U6: STM32F103C8Tx BLUEPILL, Package_QFP:LQFP-48_7x7mm_P0.5mm, symbol MCU_ST_STM32F1:STM32F103C8Tx
- added BLUEPILL1: ~, Module:Electrosmith_Daisy_Seed, symbol MCU_ST_STM32F1:Bluepill_STM32F103
- added C25, C27: C_Polarized, Capacitor_THT:C_Radial_D5.0mm_H5.0mm_P2.00mm, symbol Device:C_Polarized
- added C26, C28: 2.2n, Capacitor_THT:C_Disc_D4.7mm_W2.5mm_P5.00mm, symbol Device:C
- added D5, D6: D_Schottky, Diode_THT:D_DO-35_SOD27_P7.62mm_Horizontal, symbol Device:D_Schottky
- added J2, J3: Conn_01x20_Socket, Connector_PinHeader_2.54mm:PinHeader_1x20_P2.54mm_Vertical, symbol Connector:Conn_01x20_Socket
- added TP1, TP10, TP11, TP12, TP2, TP3, TP4, TP5, TP6, TP7, TP8, TP9: TestPoint, TestPoint:TestPoint_Loop_D1.80mm_Drill1.0mm_Beaded, symbol Connector:TestPoint
- added unit 2 of U1
- added unit 5 of U1
- added unit 1 of U1
- added unit 1 of U2
- added unit 5 of U2
- added unit 2 of U2
- C1: renamed from C8; footprint (none) -> Capacitor_THT:C_Disc_D4.7mm_W2.5mm_P5.00mm
- C10: renamed from C17; footprint (none) -> Capacitor_THT:C_Disc_D4.7mm_W2.5mm_P5.00mm
- C11: renamed from C10; footprint (none) -> Capacitor_THT:C_Disc_D4.7mm_W2.5mm_P5.00mm
- C12: renamed from C18; footprint (none) -> Capacitor_THT:C_Disc_D4.7mm_W2.5mm_P5.00mm
- C13: renamed from C1; footprint (none) -> Capacitor_THT:C_Disc_D4.7mm_W2.5mm_P5.00mm
- C14: renamed from C19; footprint (none) -> Capacitor_THT:C_Disc_D4.7mm_W2.5mm_P5.00mm
- C15: renamed from C2; footprint (none) -> Capacitor_THT:C_Disc_D4.7mm_W2.5mm_P5.00mm
- C16: renamed from C20; footprint (none) -> Capacitor_THT:C_Disc_D4.7mm_W2.5mm_P5.00mm
- C17: renamed from C3; footprint (none) -> Capacitor_THT:C_Disc_D4.7mm_W2.5mm_P5.00mm
- C18: renamed from C12; footprint (none) -> Capacitor_THT:C_Disc_D4.7mm_W2.5mm_P5.00mm
- C19: renamed from C21; footprint (none) -> Capacitor_THT:C_Disc_D4.7mm_W2.5mm_P5.00mm
- C2: renamed from C14; footprint (none) -> Capacitor_THT:C_Disc_D4.7mm_W2.5mm_P5.00mm
- C20: renamed from C22; footprint (none) -> Capacitor_THT:C_Disc_D4.7mm_W2.5mm_P5.00mm
- C21: renamed from C11; footprint (none) -> Capacitor_THT:C_Disc_D4.7mm_W2.5mm_P5.00mm
- C22: renamed from C23; footprint (none) -> Capacitor_THT:C_Disc_D4.7mm_W2.5mm_P5.00mm
- C23: renamed from C4; footprint (none) -> Capacitor_THT:C_Disc_D4.7mm_W2.5mm_P5.00mm
- C24, C9: footprint (none) -> Capacitor_THT:C_Disc_D4.7mm_W2.5mm_P5.00mm
- C3: renamed from C5; footprint (none) -> Capacitor_THT:C_Radial_D5.0mm_H5.0mm_P2.00mm
- C4: renamed from C6; footprint (none) -> Capacitor_THT:C_Disc_D4.7mm_W2.5mm_P5.00mm
- C5: renamed from C7; footprint (none) -> Capacitor_THT:C_Disc_D4.7mm_W2.5mm_P5.00mm
- C6: renamed from C15; footprint (none) -> Capacitor_THT:C_Disc_D4.7mm_W2.5mm_P5.00mm
- C7: renamed from C13; footprint (none) -> Capacitor_THT:C_Disc_D4.7mm_W2.5mm_P5.00mm
- C8: renamed from C16; footprint (none) -> Capacitor_THT:C_Disc_D4.7mm_W2.5mm_P5.00mm
- D1: footprint (none) -> Connector_PinHeader_2.54mm:PinHeader_1x02_P2.54mm_Vertical
- D2: renamed from D7; footprint (none) -> Connector_PinHeader_2.54mm:PinHeader_1x02_P2.54mm_Vertical
- D3: renamed from D2; footprint (none) -> LED_THT:LED_D3.0mm
- D4: renamed from D9; footprint (none) -> LED_THT:LED_D3.0mm
- D7: renamed from D3; footprint (none) -> LED_THT:LED_D3.0mm
- D8: renamed from D4; footprint (none) -> LED_THT:LED_D3.0mm
- J1: footprint (none) -> TerminalBlock_Phoenix:TerminalBlock_Phoenix_MKDS-1,5-2-5.08_1x02_P5.08mm_Horizontal
- J4: renamed from J2; footprint (none) -> TerminalBlock_Phoenix:TerminalBlock_Phoenix_MKDS-1,5-2-5.08_1x02_P5.08mm_Horizontal
- R1: renamed from R9; footprint (none) -> Resistor_THT:R_Axial_DIN0207_L6.3mm_D2.5mm_P10.16mm_Horizontal
- R10: renamed from R34; footprint (none) -> Resistor_THT:R_Axial_DIN0207_L6.3mm_D2.5mm_P10.16mm_Horizontal
- R11: renamed from R4; footprint (none) -> Connector_PinHeader_2.54mm:PinHeader_1x02_P2.54mm_Vertical
- R12: renamed from R35; footprint (none) -> Connector_PinHeader_2.54mm:PinHeader_1x02_P2.54mm_Vertical
- R13: renamed from R19; footprint (none) -> Resistor_THT:R_Axial_DIN0207_L6.3mm_D2.5mm_P10.16mm_Horizontal
- R14: renamed from R36; footprint (none) -> Resistor_THT:R_Axial_DIN0207_L6.3mm_D2.5mm_P10.16mm_Horizontal
- R15: renamed from R20; footprint (none) -> Resistor_THT:R_Axial_DIN0207_L6.3mm_D2.5mm_P10.16mm_Horizontal
- R16: renamed from R37; footprint (none) -> Resistor_THT:R_Axial_DIN0207_L6.3mm_D2.5mm_P10.16mm_Horizontal
- R17: renamed from R10; footprint (none) -> Resistor_THT:R_Axial_DIN0207_L6.3mm_D2.5mm_P10.16mm_Horizontal
- R18: renamed from R38; footprint (none) -> Resistor_THT:R_Axial_DIN0207_L6.3mm_D2.5mm_P10.16mm_Horizontal
- R19: renamed from R11; footprint (none) -> Resistor_THT:R_Axial_DIN0207_L6.3mm_D2.5mm_P10.16mm_Horizontal
- R2: renamed from R30; footprint (none) -> Resistor_THT:R_Axial_DIN0207_L6.3mm_D2.5mm_P10.16mm_Horizontal
- R20: renamed from R12; footprint (none) -> Resistor_THT:R_Axial_DIN0207_L6.3mm_D2.5mm_P10.16mm_Horizontal
- R21: renamed from R39; footprint (none) -> Resistor_THT:R_Axial_DIN0207_L6.3mm_D2.5mm_P10.16mm_Horizontal
- R22: renamed from R40; footprint (none) -> Resistor_THT:R_Axial_DIN0207_L6.3mm_D2.5mm_P10.16mm_Horizontal
- R23: renamed from R13; footprint (none) -> Resistor_THT:R_Axial_DIN0207_L6.3mm_D2.5mm_P10.16mm_Horizontal
- R24: renamed from R41; footprint (none) -> Resistor_THT:R_Axial_DIN0207_L6.3mm_D2.5mm_P10.16mm_Horizontal
- R25: renamed from R1; footprint (none) -> Resistor_THT:R_Axial_DIN0207_L6.3mm_D2.5mm_P10.16mm_Horizontal
- R26: renamed from R42; footprint (none) -> Resistor_THT:R_Axial_DIN0207_L6.3mm_D2.5mm_P10.16mm_Horizontal
- R27: renamed from R21; footprint (none) -> Resistor_THT:R_Axial_DIN0207_L6.3mm_D2.5mm_P10.16mm_Horizontal
- R28: renamed from R22; footprint (none) -> Resistor_THT:R_Axial_DIN0207_L6.3mm_D2.5mm_P10.16mm_Horizontal
- R29: renamed from R2; footprint (none) -> Resistor_THT:R_Axial_DIN0207_L6.3mm_D2.5mm_P10.16mm_Horizontal
- R3: renamed from R27; footprint (none) -> Resistor_THT:R_Axial_DIN0207_L6.3mm_D2.5mm_P10.16mm_Horizontal
- R30: renamed from R3; footprint (none) -> Resistor_THT:R_Axial_DIN0207_L6.3mm_D2.5mm_P10.16mm_Horizontal
- R31: renamed from R43; footprint (none) -> Resistor_THT:R_Axial_DIN0207_L6.3mm_D2.5mm_P10.16mm_Horizontal
- R32: renamed from R44; footprint (none) -> Resistor_THT:R_Axial_DIN0207_L6.3mm_D2.5mm_P10.16mm_Horizontal
- R33: renamed from R14; footprint (none) -> Resistor_THT:R_Axial_DIN0207_L6.3mm_D2.5mm_P10.16mm_Horizontal
- R34: renamed from R45; footprint (none) -> Resistor_THT:R_Axial_DIN0207_L6.3mm_D2.5mm_P10.16mm_Horizontal
- R35: renamed from R23; footprint (none) -> Resistor_THT:R_Axial_DIN0207_L6.3mm_D2.5mm_P10.16mm_Horizontal
- R36: renamed from R15; footprint (none) -> Resistor_THT:R_Axial_DIN0207_L6.3mm_D2.5mm_P10.16mm_Horizontal
- R37: renamed from R46; footprint (none) -> Resistor_THT:R_Axial_DIN0207_L6.3mm_D2.5mm_P10.16mm_Horizontal
- R38: renamed from R17; footprint (none) -> Resistor_THT:R_Axial_DIN0207_L6.3mm_D2.5mm_P10.16mm_Horizontal
- R39: renamed from R47; footprint (none) -> Resistor_THT:R_Axial_DIN0207_L6.3mm_D2.5mm_P10.16mm_Horizontal
- R4: renamed from R31; footprint (none) -> Resistor_THT:R_Axial_DIN0207_L6.3mm_D2.5mm_P10.16mm_Horizontal
- R40: renamed from R24; footprint (none) -> Resistor_THT:R_Axial_DIN0207_L6.3mm_D2.5mm_P10.16mm_Horizontal
- R41: renamed from R16; footprint (none) -> Resistor_THT:R_Axial_DIN0207_L6.3mm_D2.5mm_P10.16mm_Horizontal
- R42: renamed from R48; footprint (none) -> Resistor_THT:R_Axial_DIN0207_L6.3mm_D2.5mm_P10.16mm_Horizontal
- R43: renamed from R5; footprint (none) -> Resistor_THT:R_Axial_DIN0207_L6.3mm_D2.5mm_P10.16mm_Horizontal
- R44: renamed from R49; footprint (none) -> Resistor_THT:R_Axial_DIN0207_L6.3mm_D2.5mm_P10.16mm_Horizontal
- R45: renamed from R6; footprint (none) -> Resistor_THT:R_Axial_DIN0207_L6.3mm_D2.5mm_P10.16mm_Horizontal
- R46: renamed from R50; footprint (none) -> Resistor_THT:R_Axial_DIN0207_L6.3mm_D2.5mm_P10.16mm_Horizontal
- R47: renamed from R25; footprint (none) -> Resistor_THT:R_Axial_DIN0207_L6.3mm_D2.5mm_P10.16mm_Horizontal
- R48: renamed from R26; footprint (none) -> Resistor_THT:R_Axial_DIN0207_L6.3mm_D2.5mm_P10.16mm_Horizontal
- R49: renamed from R7; footprint (none) -> Resistor_THT:R_Axial_DIN0207_L6.3mm_D2.5mm_P10.16mm_Horizontal
- R5: renamed from R18; footprint (none) -> Resistor_THT:R_Axial_DIN0207_L6.3mm_D2.5mm_P10.16mm_Horizontal
- R50: renamed from R51; footprint (none) -> Resistor_THT:R_Axial_DIN0207_L6.3mm_D2.5mm_P10.16mm_Horizontal
- R51: renamed from R8; footprint (none) -> Resistor_THT:R_Axial_DIN0207_L6.3mm_D2.5mm_P10.16mm_Horizontal
- R52: footprint (none) -> Resistor_THT:R_Axial_DIN0207_L6.3mm_D2.5mm_P10.16mm_Horizontal
- R6: renamed from R32; footprint (none) -> Resistor_THT:R_Axial_DIN0207_L6.3mm_D2.5mm_P10.16mm_Horizontal
- R7: renamed from R29; footprint (none) -> Resistor_THT:R_Axial_DIN0207_L6.3mm_D2.5mm_P10.16mm_Horizontal
- R8: renamed from R33; footprint (none) -> Resistor_THT:R_Axial_DIN0207_L6.3mm_D2.5mm_P10.16mm_Horizontal
- R9: renamed from R28; footprint (none) -> Resistor_THT:R_Axial_DIN0207_L6.3mm_D2.5mm_P10.16mm_Horizontal
- RV1: renamed from RV2; footprint (none) -> Potentiometer_THT:Potentiometer_Bourns_3296W_Vertical
- RV2: renamed from RV3; footprint (none) -> Potentiometer_THT:Potentiometer_Bourns_3296W_Vertical
- RV3: renamed from RV1; footprint (none) -> Potentiometer_THT:Potentiometer_Bourns_3296W_Vertical
- RV4: footprint (none) -> Potentiometer_THT:Potentiometer_Bourns_3296W_Vertical
- U1: renamed from U2; footprint (none) -> Package_DIP:DIP-14_W7.62mm_Socket_LongPads
- U1: renamed from U7; footprint (none) -> Package_DIP:DIP-14_W7.62mm_Socket_LongPads
- U2: renamed from U12; footprint (none) -> Package_DIP:DIP-14_W7.62mm_Socket_LongPads
- U2: renamed from U13; footprint (none) -> Package_DIP:DIP-14_W7.62mm_Socket_LongPads
- U3: renamed from U10; footprint (none) -> Package_DIP:DIP-14_W7.62mm_Socket_LongPads
- U3: renamed from U5; footprint (none) -> Package_DIP:DIP-14_W7.62mm_Socket_LongPads
- U4: renamed from U1; footprint (none) -> Package_DIP:DIP-16_W7.62mm_Socket_LongPads
- U5: renamed from U11; footprint (none) -> Package_DIP:DIP-16_W7.62mm_Socket_LongPads
- renumbered D8 to D9
Connections:
- net +5V: now also BLUEPILL1.18 (5V), C25.1, C26.1, C27.1, C28.1, J2.18 (Pin_18), U1.4 (V+), U2.4 (V+)
- net Demod 1: now also U1.12 (+), U1.8, TP6.1; no longer U1.1, U1.3 (+)
- net Demod 2: now also U2.12 (+), U2.8; no longer U2.1, U2.3 (+)
- net GND: now also BLUEPILL1.19 (GND), BLUEPILL1.39 (GND), BLUEPILL1.40 (GND), C25.2, C26.2, C27.2, C28.2, J2.19 (Pin_19), J3.19 (Pin_19), J3.20 (Pin_20), TP11.1, TP12.1, U1.11 (V-), U1.3 (+), U2.11 (V-), U2.3 (+)
- net Gain control 1: now also BLUEPILL1.16 (PB8), J2.16 (Pin_16), TP4.1
- net Gain control 2: now also BLUEPILL1.26 (PA1), J3.6 (Pin_6)
- net Modulated input 1: now also U3.6, TP3.1; no longer U3.2
- net Modulated input 2: now also U3.8; no longer U3.2
- net Motor control: now also BLUEPILL1.31 (PA6), J3.11 (Pin_11)
- net STM32 Input (RX1): now also BLUEPILL1.15 (PB7), J2.15 (Pin_15), TP7.1
- net STM32 Input (RX2): now also BLUEPILL1.28 (PA3), J3.8 (Pin_8)
- net STM32 Output (TX1): now also BLUEPILL1.14 (PB6), J2.14 (Pin_14), J3.9 (Pin_9)
- net STM32 Output (TX2): now also BLUEPILL1.29 (PA4)
- net at C12.2, R21.2, R22.1: now also U3.9; no longer U3.1
- net at C24.2, R44.2, R46.2: now also U2.13 (-); no longer U2.2 (-)
- net ADC2: now reaches C10.2, C12.1, R10.2, R14.2, R18.1
- net ADC2: now also BLUEPILL1.27 (PA2), D6.2 (A), J3.7 (Pin_7), U2.7
- net at R49.1: now also U1.14; no longer U1.1
- net at R30.1, R33.1, U4.10 (SFout): now also TP5.1
- net at C1.2, R3.1, RV1.1: now also TP1.1, U1.1
- net at C1.1, D1.1 (K), R1.1: now also U1.2 (-)
- net at D7.1 (K), Q1.1 (C): now also TP9.1
- net ADC0: now reaches C11.1, C9.2, R13.2, R17.1, R9.2
- net ADC0: now also BLUEPILL1.25 (PA0), D5.2 (A), J3.5 (Pin_5), TP2.1, U1.7
- net at C23.2, R43.2, R45.2: now also U1.13 (-); no longer U1.2 (-)
- net at D9.2 (A), J4.1 (Pin_1), Q3.1 (C): now also TP10.1
- net at C9.1, R11.1, R5.2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: now also U1.6 (-)
- net at C2.1, D2.1 (K), R2.1: now also U2.2 (-)
- net at R38.2, R41.1: now also U1.9 (-); no longer U1.2 (-)
- net at C10.1, R12.1, R6.2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: now also U2.6 (-)
- net at C8.2, R8.2: now also U2.5 (+)
- net at C2.2, R4.1, RV2.1: now also U2.1
- net at C11.2, R19.2, R20.1: now also U3.5; no longer U3.1
- net at R37.2: now also U2.10 (+); no longer U2.3 (+)
- net at C7.2, R7.2: now also U1.5 (+)
- net at R36.2: now also U1.10 (+); no longer U1.3 (+)
- net at R50.1: now also U2.14; no longer U2.1
- net at Q1.2 (B), R28.2: now also TP8.1
- net at R39.2, R42.1: now also U2.9 (-); no longer U2.2 (-)
- new net +3.3V: BLUEPILL1.20 (3V3), BLUEPILL1.38 (3V3), D5.1 (K), D6.1 (K), J2.20 (Pin_20), J3.18 (Pin_18)
- new net NRST: BLUEPILL1.37 (NRST), J3.17 (Pin_17)
- new net PA10: BLUEPILL1.7 (PA10), J2.7 (Pin_7)
- new net PA11: BLUEPILL1.8 (PA11), J2.8 (Pin_8)
- new net PA12: BLUEPILL1.9 (PA12), J2.9 (Pin_9)
- new net PA15: BLUEPILL1.10 (PA15), J2.10 (Pin_10)
- new net PA5: BLUEPILL1.30 (PA5), J3.10 (Pin_10)
- new net PA7: BLUEPILL1.32 (PA7), J3.12 (Pin_12)
- new net PA8: BLUEPILL1.5 (PA8), J2.5 (Pin_5)
- new net PA9: BLUEPILL1.6 (PA9), J2.6 (Pin_6)
- new net PB0: BLUEPILL1.33 (PB0), J3.13 (Pin_13)
- new net PB1: BLUEPILL1.34 (PB1), J3.14 (Pin_14)
- new net PB10: BLUEPILL1.35 (PB10), J3.15 (Pin_15)
- new net PB11: BLUEPILL1.36 (PB11), J3.16 (Pin_16)
- new net PB12: BLUEPILL1.1 (PB12), J2.1 (Pin_1)
- new net PB13: BLUEPILL1.2 (PB13), J2.2 (Pin_2)
- new net PB14: BLUEPILL1.3 (PB14), J2.3 (Pin_3)
- new net PB15: BLUEPILL1.4 (PB15), J2.4 (Pin_4)
- new net PB3: BLUEPILL1.11 (PB3), J2.11 (Pin_11)
- new net PB4: BLUEPILL1.12 (PB4), J2.12 (Pin_12)
- new net PB5: BLUEPILL1.13 (PB5), J2.13 (Pin_13)
- new net PB9: BLUEPILL1.17 (PB9), J2.17 (Pin_17)
- new net PC13: BLUEPILL1.22 (PC13), J3.2 (Pin_2)
- new net PC14: BLUEPILL1.23 (PC14), J3.3 (Pin_3)
- new net PC15: BLUEPILL1.24 (PC15), J3.4 (Pin_4)
- new net VBAT: BLUEPILL1.21 (VBAT), J3.1 (Pin_1)
Other:
- note added: "TRANSIMPEDANCE AMPLIFIER"
- note removed: "TRANSINPEDANCE AMPLIFIER"
- moved on the sheet: C3, C4, D7, J1, Q3, R48
