File: proj_td3/proj_td3.kicad_pcb (KiCad board)
At the start: 2 copper layers, 115.6 x 45.7 mm, 78 parts, among them J1 Motor, J2 Input 5V, J3 Conn_01x20_Socket, J4 Conn_01x20_Socket, J5 Conn_01x04_Pin, Q1 BC546, Q2 BC546, Q3 BC546, U1 4066, U2 LM358, U3 LM358

Commit message: avances proj td3
Parts:
- removed C5: C_Polarized, Capacitor_THT:C_Radial_D5.0mm_H5.0mm_P2.00mm
- removed C6: 2.2n, Capacitor_THT:C_Disc_D4.7mm_W2.5mm_P5.00mm
- removed J5: Conn_01x04_Pin, Connector_PinHeader_2.54mm:PinHeader_1x04_P2.54mm_Vertical
- removed Q1: BC546, Package_TO_SOT_THT:TO-92_Inline
- removed TP22, TP23: TestPoint, TestPoint:TestPoint_THTPad_1.0x1.0mm_Drill0.5mm
- added JP3: Jumper_2_Open, Connector_PinHeader_2.54mm:PinHeader_1x02_P2.54mm_Vertical, B.Cu at (34.9, 23.0)
- added Q4: TIP122, Package_TO_SOT_THT:TO-220-3_Vertical, B.Cu at (111.1, 72.3)
- added RV5: 10k, Potentiometer_THT:Potentiometer_Bourns_3296W_Vertical, B.Cu at (31.2, 61.2)
- added RV6: 10k, Potentiometer_THT:Potentiometer_Bourns_3296W_Vertical, B.Cu at (31.2, 71.5)
- D1, D2, D3, Q2, Q3, R1, R2, R3, R5, TP1, TP10, TP2, TP3, TP4, TP5, TP6, TP7, TP8, TP9: moved to B.Cu
- J1, J2: footprint TerminalBlock_Phoenix:TerminalBlock_Phoenix_MKDS-1,5-2-5.08_1x02_P5.08mm_Horizontal -> TerminalBlock_Phoenix:TerminalBlock_Phoenix_MPT-0,5-2-2.54_1x02_P2.54mm_Horizontal; moved to B.Cu
- R4, R6: value 22k -> 1k; moved to B.Cu
- moved C8 592.8 mm to (57.0, 71.0), turned to 0 degrees
- moved C7 583.2 mm to (65.7, 71.6), turned to 0 degrees
- moved J2 543.2 mm to (49.9, 72.9)
- moved TP10 542.3 mm to (42.9, 50.7), turned to 180 degrees
- moved TP1 535.3 mm to (72.8, 71.6), turned to -90 degrees
- moved TP2 531.3 mm to (77.4, 71.6), turned to -90 degrees
- moved TP3 527.4 mm to (82.1, 71.6), turned to -90 degrees
- moved TP4 511.0 mm to (87.4, 71.6), turned to 180 degrees
- moved TP6 509.4 mm to (41.7, 27.2), turned to 180 degrees
- moved TP5 507.8 mm to (92.5, 71.6), turned to 180 degrees
- moved D2 507.4 mm to (30.0, 44.0), turned to 90 degrees
- moved R2 499.3 mm to (96.3, 71.6)
- moved R3 487.5 mm to (49.3, 23.4), turned to 180 degrees
- moved D1 476.8 mm to (124.6, 69.2), turned to 180 degrees
- moved Q2 475.4 mm to (55.6, 25.9), turned to 90 degrees
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Routing:
- net +5V: track 17.5 -> 267.3 mm, vias 0 -> 5
- net ADC4 (Muestreo FSK 2): track 71.2 -> 137.7 mm, vias 1 -> 2
- net GND: track 63.3 -> 110.2 mm, vias 0 -> 1
- net Net-(D1-A): track 0.00 -> 46.4 mm
- net T4C4 (Señal LED FSK 1): track 6.35 -> 48.3 mm, vias 0 -> 1
- net Net-(D2-K): track 0.00 -> 41.0 mm
- net Net-(Q2-B): track 0.00 -> 36.9 mm
- net Net-(D3-K): track 0.00 -> 36.9 mm
- net ADC5 (Muestreo FSK 1): track 52.8 -> 84.6 mm
- net Net-(D5-K): track 121.4 -> 91.2 mm
- net Net-(R17-Pad1): track 64.7 -> 36.9 mm
- net Net-(R16-Pad1): track 52.9 -> 28.0 mm
- net Net-(D2-A): track 0.00 -> 21.9 mm
- net Net-(Q3-B): track 0.00 -> 21.2 mm
- net Net-(Q4-B): track 0.00 -> 20.5 mm
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- added copper zone on F.Cu, net GND
Other:
- board size 115.6 x 45.7 mm -> 120.5 x 55.9 mm
- board text added: "UTN TD3 511 2023"
- board text added: "VELAZQUEZ ALAN"
