File: proj_td3/proj_td3.kicad_sch (KiCad schematic)
At the start: 72 parts, among them J1 Input 5V, J2 Conn_01x20_Socket, J3 Conn_01x20_Socket, J4 Motor, J5 Conn_01x04_Pin, Q1 BC546, Q3 BC546, U1 4066, U2 LM358, U3 LM358

Commit message: proj td3 avances
Parts:
- added JP1, JP2: SolderJumper_3_Open, symbol Jumper:SolderJumper_3_Open
- BLUEPILL1: footprint Module:Electrosmith_Daisy_Seed -> Package_SO:SO-14_5.3x10.2mm_P1.27mm
- TP10, TP11, TP12, TP13, TP14, TP15, TP16, TP17, TP18, TP19, TP20, TP21, TP22, TP23: footprint (none) -> TestPoint:TestPoint_THTPad_1.0x1.0mm_Drill0.5mm
- TP5: footprint (none) -> TestPoint:TestPoint_Loop_D1.80mm_Drill1.0mm_Beaded
- U1: footprint (none) -> Package_SO:SO-14_5.3x10.2mm_P1.27mm
- U2, U3: footprint (none) -> Package_SO:SO-8_5.3x6.2mm_P1.27mm
Connections:
- net ADC4 (Muestreo FSK 2): now also JP1.1 (A)
- net ADC5 (Muestreo FSK 1): now also JP2.1 (A)
- net at C4.2, R18.2, TP19.1: now also JP1.2 (C); no longer U3.5 (+)
- net at C2.2, R10.2, TP13.1: now also JP2.2 (C); no longer U2.5 (+)
- new net: JP2.3 (B), U2.5 (+)
- new net: JP1.3 (B), U3.5 (+)

Commit message: avances proyecto td3
Parts:
- removed U1: LM324, Package_DIP:DIP-14_W7.62mm_Socket_LongPads, symbol Amplifier_Operational:LM324
- added C25: C_Polarized, Capacitor_THT:C_Radial_D5.0mm_H5.0mm_P2.00mm, symbol Device:C_Polarized
- added C26: 2.2n, Capacitor_THT:C_Disc_D4.7mm_W2.5mm_P5.00mm, symbol Device:C
- added unit 3 of U3
- BLUEPILL1: footprint Package_SO:SO-14_5.3x10.2mm_P1.27mm -> Module:Electrosmith_Daisy_Seed
- C1, C2, C3, C4: footprint (none) -> Capacitor_THT:C_Disc_D3.0mm_W2.0mm_P2.50mm
- D4, D5: footprint (none) -> Connector_PinHeader_2.54mm:PinHeader_1x02_P2.54mm_Vertical
- J5: footprint (none) -> Connector_PinHeader_2.54mm:PinHeader_1x04_P2.54mm_Vertical
- JP1, JP2: footprint (none) -> Jumper:SolderJumper-3_P1.3mm_Open_RoundedPad1.0x1.5mm
- R10, R11, R12, R13, R14, R15, R16, R17, R18, R19, R20, R21, R22, R7, R8, R9: footprint (none) -> Resistor_THT:R_Axial_DIN0207_L6.3mm_D2.5mm_P10.16mm_Horizontal
- RV1, RV2, RV3, RV4: footprint (none) -> Potentiometer_THT:Potentiometer_Bourns_3296W_Vertical
Connections:
- net +5V: now also C25.1, C26.1, U3.8 (V+)
- net GND: now also C25.2, C26.2, U3.4 (V-)
Other:
- moved on the sheet: C25, C26, U1E, U2C

Commit message: avances proj td3
Parts:
- removed C25: C_Polarized, Capacitor_THT:C_Radial_D5.0mm_H5.0mm_P2.00mm, symbol Device:C_Polarized
- removed C26: 2.2n, Capacitor_THT:C_Disc_D4.7mm_W2.5mm_P5.00mm, symbol Device:C
- removed J5: Conn_01x04_Pin, Connector_PinHeader_2.54mm:PinHeader_1x04_P2.54mm_Vertical, symbol Connector:Conn_01x04_Pin
- removed Q3: BC546, Package_TO_SOT_THT:TO-92_Inline, symbol Transistor_BJT:BC546
- removed TP22, TP23: TestPoint, TestPoint:TestPoint_THTPad_1.0x1.0mm_Drill0.5mm, symbol Connector:TestPoint
- added JP3: Jumper_2_Open, Connector_PinHeader_2.54mm:PinHeader_1x02_P2.54mm_Vertical, symbol Jumper:Jumper_2_Open
- added Q4: TIP122, Package_TO_SOT_THT:TO-220-3_Vertical, symbol Transistor_BJT:TIP122
- added RV5, RV6: 10k, Potentiometer_THT:Potentiometer_Bourns_3296W_Vertical, symbol Device:R_Potentiometer_Trim
- J1, J4: footprint TerminalBlock_Phoenix:TerminalBlock_Phoenix_MKDS-1,5-2-5.08_1x02_P5.08mm_Horizontal -> TerminalBlock_Phoenix:TerminalBlock_Phoenix_MPT-0,5-2-2.54_1x02_P2.54mm_Horizontal
- R28: value 22k -> 1k
Connections:
- net ADC8 (Seteo distancia): now also RV6.3
- net ADC9 (Seteo velocidad): now also RV5.3
- net EXT IT (Input modo): now also JP3.1 (A)
- net GND: now also JP3.2 (B), Q4.3 (E), RV5.1, RV5.2, RV6.1, RV6.2
- net at D9.2 (A), J4.1 (Pin_1), TP10.1: now also Q4.2 (C)
- net at R48.2, TP5.1: now also Q4.1 (B)
Other:
- note added: "CORREGIR!!!"
- moved on the sheet: C25, C26, U3C
